File: Smart_Trainer_Kit_v1/v1_pcb_project_files.kicad_sch (KiCad schematic)
At the start: 96 parts, among them SW1 SW_DIP_x01, SW10 SW_DIP_x01, SW2 SW_DIP_x01, SW3 SW_DIP_x01, SW4 SW_DIP_x01, SW5 SW_DIP_x01, SW6 SW_DIP_x01, SW7 SW_DIP_x01, SW8 SW_DIP_x01, SW9 SW_DIP_x01, U1 CD4511B, U2 D168K, U3 lm2596 buck boost, U4 LM741

Commit message: cleaned uo
Parts:
- removed D11, D12: CQY99, LED_THT:LED_D5.0mm_IRGrey, symbol LED:CQY99
- removed R11, R12: 330, Resistor_THT:R_Axial_DIN0204_L3.6mm_D1.6mm_P7.62mm_Horizontal, symbol Device:R_US
- removed SW1, SW10, SW2, SW3, SW4, SW5, SW6, SW7, SW8, SW9: SW_DIP_x01, Button_Switch_THT:SW_CW_GPTS203211B, symbol Switch:SW_DIP_x01
- removed U3: lm2596 buck boost, DC_DC_LM2596_small:DC_DC_LM2596_small, symbol 4xxx:4023
- added R23: 330, Resistor_THT:R_Axial_DIN0207_L6.3mm_D2.5mm_P7.62mm_Horizontal, symbol Device:R_US
- added SW1, SW10, SW2, SW3, SW4, SW5, SW6, SW7, SW8, SW9: SW_Push_SPDT, Button_Switch_THT:SPDT_platemount_switch(platemount), symbol Switch:SW_Push_SPDT
- BP18, BP19, BP20, BP21, BP22, BP23, BP24, BP25, BP26, BP27, BP28, BP29, BP30, BP31, BP32, BP33, BP34, BP35, BP36, BP37, BP38, BP39, BP40, BP41, BP42, BP43, BP44: footprint (none) -> MountingHole:banana_plug(modified thickness)
- BP28: renamed from AE1; value Antenna -> banana plug; footprint (none) -> MountingHole:banana_plug(modified thickness)
- BP29: renamed from AE2; value Antenna -> banana plug; footprint (none) -> MountingHole:banana_plug(modified thickness)
- BP30: renamed from AE3; value Antenna -> banana plug; footprint (none) -> MountingHole:banana_plug(modified thickness)
- D1, D10, D13, D14, D15, D16, D17, D18, D19, D2, D20, D22, D23, D24, D3, D4, D5, D6, D7, D8, D9: footprint LED_THT:LED_D5.0mm_IRGrey -> LED_THT:LED_D3.0mm
- R1, R10, R13, R14, R15, R16, R17, R18, R19, R2, R20, R21, R22, R23, R3, R4, R5, R6, R7, R8, R9: footprint Resistor_THT:R_Axial_DIN0204_L3.6mm_D1.6mm_P7.62mm_Horizontal -> Resistor_THT:R_Axial_DIN0207_L6.3mm_D2.5mm_P7.62mm_Horizontal
- U1: footprint Socket:DIP_Socket-16_W4.3_W5.08_W7.62_W10.16_W10.9_3M_216-3340-00-0602J -> Package_DIP:DIP-16_W7.62mm_Socket_LongPads
Connections:
- net VDD is gone; now on net +5V: U1.3 (~{LT}), U1.4 (~{BI})
- net +5V: now also A1.5 (+5V), BP23.1 (A), SW1.1 (A), SW10.1 (A), SW2.1 (A), SW3.1 (A), SW4.1 (A), SW5.1 (A), SW6.1 (A), SW7.1 (A), SW8.1 (A), SW9.1 (A)
- net GNDREF: now also A1.29 (GND), BP22.1 (A), R23.2, SW1.3 (C), SW10.3 (C), SW2.3 (C), SW3.3 (C), SW4.3 (C), SW5.3 (C), SW6.3 (C), SW7.3 (C), SW8.3 (C), SW9.3 (C)
- net V(input): now also R23.1
- net at BP38.1 (A), D7.2 (A): now also SW7.2 (B)
- net at BP41.1 (A), D10.2 (A): now also SW10.2 (B)
- net at BP34.1 (A), D3.2 (A): now also SW3.2 (B)
- net at BP37.1 (A), D6.2 (A): now also SW6.2 (B)
- net at BP39.1 (A), D8.2 (A): now also SW8.2 (B)
- net at BP36.1 (A), D5.2 (A): now also SW5.2 (B)
- net at BP35.1 (A), D4.2 (A): now also SW4.2 (B)
- net at BP33.1 (A), D2.2 (A): now also SW2.2 (B)
- net at BP40.1 (A), D9.2 (A): now also SW9.2 (B)
- net at BP32.1 (A), D1.2 (A): now also SW1.2 (B)
Other:
- moved on the sheet: BP23
